File: PCB/Ikea Chandelier.sch (KiCad schematic (older format))
At the start: 22 parts, among them J1 Arduino_Pro_Mini_Header, P1 RGB12, P2 Power, P3 RGB34, P4 RS485, P5 RGB56, P6 Candles, U1 78L05, U2 MAX485

Commit message: SMD jumper + code testing
Parts:
- JP1: footprint Pin_Headers:Pin_Header_Straight_1x02 -> septillion_device:SMD_jumper2
Connections:
- net at J1.24 (RAW): now also JP1.1
Changed lines of the file:
@@
 F 0 "JP1" H 5750 3180 50  0000 C CNN
 F 1 "Jumper_NC_Small" H 5760 3040 50  0001 C CNN
-F 2 "Pin_Headers:Pin_Header_Straight_1x02" H 5750 3100 50  0001 C CNN
+F 2 "septillion_device:SMD_jumper2" H 5750 3100 50  0001 C CNN
 F 3 "" H 5750 3100 50  0000 C CNN
 	1    5750 3100
